File: Keynux.kicad_pcb (KiCad board)
At the start: 2 copper layers, 181 parts, among them U3 Nice_Nano_V2

Commit message: connected everything, now connect to mc
Parts:
- moved D28 38.1 mm to (707.5, 25.4)
- moved S28 38.1 mm to (698.0, 22.6)
- moved D15 19.1 mm to (745.6, 25.4)
- moved S15 19.1 mm to (736.1, 22.6)
- moved D14 19.0 mm to (726.5, 25.4)
- moved S14 19.0 mm to (717.0, 22.6)
- moved U3 1.17 mm to (764.6, 29.7)
Connections:
- U3 pad 1: Row 1 -> (no net)
- U3 pad 10: Col 1 -> (no net)
- U3 pad 11: Col 2 -> (no net)
- U3 pad 12: Col 3 -> (no net)
- U3 pad 13: Col 4 -> (no net)
- U3 pad 14: Col 5 -> (no net)
- U3 pad 15: Col 6 -> (no net)
- U3 pad 16: Col 7 -> (no net)
- U3 pad 17: Col 8 -> (no net)
- U3 pad 18: Col 9 -> (no net)
- U3 pad 19: Col 10 -> (no net)
- U3 pad 2: Row 0 -> (no net)
- U3 pad 20: Col 11 -> (no net)
- U3 pad 21: unconnected-(U3-3.3v-Pad21) -> (no net)
- U3 pad 22: unconnected-(U3-RST-Pad22) -> (no net)
- U3 pad 23: unconnected-(U3-GND-Pad23) -> (no net)
- U3 pad 24: unconnected-(U3-B+-Pad24) -> (no net)
- U3 pad 25: Col 12 -> (no net)
- U3 pad 26: Col 13 -> (no net)
- U3 pad 27: Col 14 -> (no net)
- U3 pad 3: unconnected-(U3-GND-Pad3) -> (no net)
- U3 pad 4: unconnected-(U3-GND-Pad4) -> (no net)
- U3 pad 5: Row 2 -> (no net)
- U3 pad 6: Row 3 -> (no net)
- U3 pad 7: Row 4 -> (no net)
- U3 pad 8: Row 5 -> (no net)
- U3 pad 9: Col 0 -> (no net)
Routing:
- net Col 3: track 0.00 -> 301.2 mm, vias 0 -> 2
- net Col 4: track 0.00 -> 282.2 mm, vias 0 -> 2
- net Col 6: track 0.00 -> 237.9 mm, vias 0 -> 2
- net Col 14: track 0.00 -> 214.4 mm, vias 0 -> 2
- net Col 7: track 0.00 -> 214.2 mm, vias 0 -> 2
- net Col 13: track 0.00 -> 203.2 mm, vias 0 -> 2
- net Col 11: track 0.00 -> 172.9 mm
- net Col 10: track 0.00 -> 168.0 mm
- net Col 9: track 0.00 -> 164.9 mm
- net Col 8: track 0.00 -> 149.2 mm
- net Col 12: track 0.00 -> 135.4 mm
- net Col 5: track 0.00 -> 134.8 mm
- net Col 2: track 0.00 -> 123.6 mm
- net Col 1: track 0.00 -> 121.5 mm
- net Col 0: track 0.00 -> 111.7 mm
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
Commit message: update
Connections:
- U3 pad 1: (no net) -> Row 1
- U3 pad 10: (no net) -> Col 1
- U3 pad 11: (no net) -> Col 2
- U3 pad 12: (no net) -> Col 3
- U3 pad 13: (no net) -> Col 4
- U3 pad 14: (no net) -> Col 5
- U3 pad 15: (no net) -> Col 6
- U3 pad 16: (no net) -> Col 7
- U3 pad 17: (no net) -> Col 8
- U3 pad 18: (no net) -> Col 9
- U3 pad 19: (no net) -> Col 10
- U3 pad 2: (no net) -> Row 0
- U3 pad 20: (no net) -> Col 11
- U3 pad 21: (no net) -> unconnected-(U3-3.3v-Pad21)
- U3 pad 22: (no net) -> unconnected-(U3-RST-Pad22)
- U3 pad 23: (no net) -> unconnected-(U3-GND-Pad23)
- U3 pad 24: (no net) -> unconnected-(U3-B+-Pad24)
- U3 pad 25: (no net) -> Col 12
- U3 pad 26: (no net) -> Col 13
- U3 pad 27: (no net) -> Col 14
- U3 pad 3: (no net) -> unconnected-(U3-GND-Pad3)
- U3 pad 4: (no net) -> unconnected-(U3-GND-Pad4)
- U3 pad 5: (no net) -> Row 2
- U3 pad 6: (no net) -> Row 3
- U3 pad 7: (no net) -> Row 4
- U3 pad 8: (no net) -> Row 5
- U3 pad 9: (no net) -> Col 0
Routing:
- net Col 0: track 111.7 -> 504.9 mm
- net Col 1: track 121.5 -> 489.9 mm, vias 0 -> 3
- net Col 3: track 301.2 -> 626.0 mm, vias 2 -> 5
- net Row 4: track 339.0 -> 522.7 mm
- net Row 5: track 434.7 -> 597.3 mm
- net Row 3: track 326.8 -> 468.3 mm
- net Row 2: track 347.7 -> 461.4 mm
- net Col 12: track 135.4 -> 245.4 mm, vias 0 -> 1
- net Col 13: track 203.2 -> 290.7 mm, vias 2 -> 3
- net Row 1: track 377.6 -> 460.2 mm
- net Col 14: track 214.4 -> 276.6 mm, vias 2 -> 3
- net Col 2: track 123.6 -> 150.5 mm
- net Row 0: track 334.3 -> 351.6 mm

Commit message: save
Parts:
- moved D11 376.5 mm to (264.6, 39.7)
- moved D23 376.5 mm to (169.3, 68.3)
- moved D26 376.5 mm to (226.5, 68.3)
- moved D38 376.5 mm to (178.9, 87.7)
- moved D40 376.5 mm to (217.0, 87.3)
- moved D51 376.5 mm to (145.5, 106.4)
- moved D54 376.5 mm to (202.7, 106.4)
- moved D56 376.5 mm to (240.8, 106.4)
- moved D59 376.5 mm to (264.6, 68.3)
- moved D67 376.5 mm to (157.4, 125.5)
- moved D7 376.5 mm to (178.9, 39.7)
- moved D70 376.5 mm to (214.6, 125.5)
- moved D72 376.5 mm to (252.7, 125.5)
- moved D80 376.5 mm to (300.3, 96.9)
- moved D81 376.5 mm to (157.4, 144.5)
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Routing:
- net Col 4: track 282.2 -> 601.5 mm, vias 2 -> 4
- net Col 2: track 150.5 -> 443.1 mm, vias 0 -> 1
- net Col 5: track 134.8 -> 405.7 mm, vias 0 -> 2
- net Col 6: track 237.9 -> 490.2 mm, vias 2 -> 4
- net Col 7: track 214.2 -> 449.8 mm, vias 2 -> 4
- net Col 8: track 149.2 -> 364.2 mm, vias 0 -> 2
- net Col 9: track 164.9 -> 357.3 mm, vias 0 -> 2
- net Col 10: track 168.0 -> 336.9 mm, vias 0 -> 2
- net Col 11: track 172.9 -> 321.3 mm, vias 0 -> 2
- added copper zone on B.Cu, net (none)
- added copper zone on F.Cu, net (none)
Other:
- board outline added: 390.5 x 133.4 mm
- board text added: "Keynux 90"
